File: Mark_III/RGB_Amp_Internal/Kicad/Sega_MarkIII_RGB_Amp_Internal.kicad_pcb (KiCad board)
At the start: 2 copper layers, 28.6 x 19.7 mm, 12 parts, among them IC1 THS7314D, J1 RGBS Input, J2 RGBS Output

Commit message: Redesigned PCB
Other:
- board text added: "1 = GND (DIN p2) 2 = BLUE (DIN p8) 3 = GREEN (DIN p5) 4 = RED (DIN p6) 5 = SYNC (DIN p7)"
- board text removed: "1 = GND (DIN p2) 2 = BLUE (DIN p8) 3 = GREEN (DIN p4) 4 = RED (DIN p7) 5 = SYNC (DIN p6)"
