File: Mark_III/RGB_Amp_Internal/Kicad/Sega_MarkIII_RGB_Amp_Internal.kicad_sch (KiCad schematic)
At the start: 13 parts, among them IC1 THS7314D, J1 RGBS Input, J2 RGBS Output, J3 RGBS Output

Commit message: Redesigned PCB
Connections:
- net GREEN_{OUT}: now also J3.5; no longer J3.4
- net RED_{OUT}: now also J3.6; no longer J3.7
- net SYNC_{OUT}: now also J3.7; no longer J3.6
Other:
- note added: "+5V"
- note added: "Audio"
- note added: "Video"
- moved on the sheet: C1, H1, IC1, J1, J2, R1, R2, R3, R4, R5, R6, R7
