File: Saturn/Keyboard/KiCad/Sega_Saturn_Keyboard.kicad_pcb (KiCad board)
At the start: 2 copper layers, 88 parts, among them SW1 RH CTRL, SW10 PRINT SCREEN, SW11 SCROLL LOCK, SW12 PAUSE, SW13 ? /, SW14 _ \, SW15 UP, SW16 LEFT, SW17 DOWN, SW18 RIGHT, SW19 PAGE DOWN, SW2 LH CTRL, SW20 PAGE UP, SW21 > ., SW22 無変換, SW23 カタカナ, SW24 前候補, SW25 SPACE, SW26 Z, SW27 END, SW28 K, SW29 L, SW3 RH SHIFT, SW30 + ;, SW31 * :, SW32 } ], SW33 ENTER, SW34 X, SW35 HOME, SW36 I, SW37 O, SW38 P, SW39 ' @, SW4 LH SHIFT, SW40 { [, SW41 DELETE, SW42 A, SW43 INSERT, SW44 ( 8, SW45 ) 9, SW46 ~ 0, SW47 = -, SW48 _ ^, SW49 | ¥, SW5 F8, SW50 S, SW51 BACKSPACE, SW52 < ,, SW53 M, SW54 N, SW55 B, SW56 V, SW57 C, SW58 J, SW59 H, SW6 F9, SW60 G, SW61 F, SW62 D, SW63 CAPS LOCK, SW64 U, SW65 Y, SW66 T, SW67 R, SW68 W, SW69 TAB, SW7 F10, SW70 E, SW71 半角/全角, SW72 ' 7, SW73 & 6, SW74 % 5, SW75 $ 4, SW76 # 3, SW77 " 2, SW78 Q, SW79 ! 1, SW8 F11, SW80 F7, SW81 F6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

Commit message: Initial PCB routing completed
Parts:
- added C1: 10µF, Capacitor_THT:CP_Radial_D8.0mm_P2.50mm, F.Cu at (334.0, 99.3)
- added CN1: Saturn, Connector_Dsub:DSUB-9_Pins_Horizontal_P2.77x2.84mm_EdgePinOffset7.70mm_Housed_MountingHolesOffset9.12mm, F.Cu at (430.8, 88.0)
- added H1: MountingHole, MountingHole:MountingHole_3.2mm_M3, F.Cu at (445.8, 81.3)
- added H2: MountingHole, MountingHole:MountingHole_3.2mm_M3, F.Cu at (85.8, 81.3)
- added H3: MountingHole, MountingHole:MountingHole_3.2mm_M3, F.Cu at (249.8, 81.3)
- added H4: MountingHole, MountingHole:MountingHole_3.2mm_M3, F.Cu at (265.8, 234.3)
- added H5: MountingHole, MountingHole:MountingHole_3.2mm_M3, F.Cu at (445.8, 234.3)
- added H6: MountingHole, MountingHole:MountingHole_3.2mm_M3, F.Cu at (85.8, 234.3)
- added RN1: 10KΩ, Resistor_THT:R_Array_SIP9, F.Cu at (323.8, 99.3)
- added RN2: R_Network07, Resistor_THT:R_Array_SIP8, F.Cu at (364.5, 99.3)
- added SW84: F3, PCM_Switch_Keyboard_Cherry_MX:SW_Cherry_MX_PCB_1.00u, F.Cu at (175.2, 114.5)
- added U1: Teensy4.1, Clueless_Engineer:Teensy41, F.Cu at (292.1, 86.6)
- renumbered SW84 to SW85, SW85 to SW86, SW86 to SW87, SW87 to SW88, SW88 to SW89
Routing:
- net /COL 17: track 0.00 -> 974.1 mm
- net /COL 21: track 0.00 -> 838.4 mm
- net /COL 18: track 0.00 -> 768.7 mm
- net /COL 19: track 0.00 -> 624.7 mm
- net /COL 20: track 0.00 -> 571.9 mm
- net /ROW 14: track 0.00 -> 532.2 mm
- net /COL 22: track 0.00 -> 369.8 mm
- net /ROW 5: track 313.4 -> 639.2 mm
- net /COL 16: track 678.1 -> 955.8 mm
- net /COL 23: track 0.00 -> 256.7 mm
- net /ROW 9: track 0.00 -> 212.4 mm
- net /ROW 7: track 361.4 -> 573.6 mm
- net /GND: track 0.00 -> 208.1 mm
- net /+5V_{OUT}: track 0.00 -> 203.2 mm
- net /ROW 6: track 332.0 -> 511.3 mm
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Other:
- board outline added: 368 x 161 mm

Commit message: Additional text on PCB
Parts:
- RN2: value R_Network07 -> 100KΩ
- moved H1 4.50 mm to (445.8, 76.8)
- moved H2 4.50 mm to (85.8, 76.8)
- moved H3 4.50 mm to (249.8, 76.8)
- moved CN1 4.41 mm to (430.4, 83.6)
Routing:
- net /+5V_{OUT}: track 203.2 -> 207.4 mm
- net /U_{D0}: track 126.7 -> 131.0 mm
- net /L_{D2}: track 125.4 -> 129.7 mm
- net /TH_{S0}: track 118.2 -> 122.5 mm
- net /TR_{S1}: track 111.5 -> 115.7 mm
- net /TL: track 143.4 -> 147.6 mm
- net /R_{D3}: track 133.9 -> 138.2 mm
- net /D_{D1}: track 135.3 -> 139.4 mm
- net /GND: track 208.1 -> 208.5 mm, vias 0 -> 33
- added copper zone on B.Cu, net /GND
- added copper zone on F.Cu, net /GND
Other:
- board size 368 x 161 mm -> 368 x 165.5 mm
- board text added: "Brett Hallen, Dec 2025"
- board text added: "セガサターンキーボード Sega Saturn Keyboard"

Commit message: Swapped DE9 male -> female
Parts:
- CN1: footprint Connector_Dsub:DSUB-9_Pins_Horizontal_P2.77x2.84mm_EdgePinOffset7.70mm_Housed_MountingHolesOffset9.12mm -> Connector_Dsub:DSUB-9_Socket_Horizontal_P2.77x2.84mm_EdgePinOffset7.70mm_Housed_MountingHolesOffset9.12mm
- moved CN1 11.1 mm to (419.3, 83.7)
Connections:
- RN2 pad 2: /TL -> /TR_{S1}
- RN2 pad 3: /D_{D1} -> /TH_{S0}
- RN2 pad 4: /R_{D3} -> /L_{D2}
- RN2 pad 6: /L_{D2} -> /R_{D3}
- RN2 pad 7: /TH_{S0} -> /D_{D1}
- RN2 pad 8: /TR_{S1} -> /TL
- U1 pad 25: /TR_{S1} -> /TL
- U1 pad 26: /TH_{S0} -> /D_{D1}
- U1 pad 27: /L_{D2} -> /R_{D3}
- U1 pad 29: /R_{D3} -> /L_{D2}
- U1 pad 30: /D_{D1} -> /TH_{S0}
- U1 pad 31: /TL -> /TR_{S1}
Routing:
- net /TR_{S1}: track 115.7 -> 145.2 mm
- net /TL: track 147.6 -> 120.2 mm
- net /TH_{S0}: track 122.5 -> 139.4 mm
- net /D_{D1}: track 139.4 -> 122.5 mm
- net /+5V_{OUT}: track 207.4 -> 193.5 mm
- net /R_{D3}: track 138.2 -> 129.7 mm
- net /L_{D2}: track 129.7 -> 138.2 mm
- net /GND: track 208.5 -> 207.5 mm

Commit message: Design tweaks
Routing:
- net /GND: track 207.5 -> 210.1 mm
